Commit message: feat: new camera mount

File: src/ur3e_hande_robot_description/urdf/camera_mount.xacro (robot description, xacro)
@@ -74,5 +74,5 @@
     <parent link="mount" />
     <child link="camera_base" />
-    <origin xyz="0. -0.09 0.0725" rpy="${pi/2} 0. 0." />
+    <origin xyz="0. -0.11 0.0725" rpy="${pi/2} 0. 0." />
   </joint>
   <joint name="camera_base_to_camera_base_map" type="fixed">
