Commit message: fix: xacro

File: src/custom-ur-descriptions/ur3e_hande_robot_description/urdf/ur_with_hande.xacro (robot description, xacro)
@@ -12,8 +12,8 @@
    <!-- These parameters are from https://github.com/UniversalRobots/Universal_Robots_ROS2_Description/blob/29e90d5095fdf4af99eba3c3eae153d7d5d769c0/urdf/ur.urdf.xacro-->
    <xacro:arg name="tf_prefix" default="" />
-   <xacro:arg name="joint_limit_params" default="$(find ur_description)/config/$(arg ur_type)/joint_limits.yaml"/>
-   <xacro:arg name="kinematics_params" default="$(find ur_description)/config/$(arg ur_type)/default_kinematics.yaml"/>
-   <xacro:arg name="physical_params" default="$(find ur_description)/config/$(arg ur_type)/physical_parameters.yaml"/>
-   <xacro:arg name="visual_params" default="$(find ur_description)/config/$(arg ur_type)/visual_parameters.yaml"/>
+   <xacro:property name="joint_limit_params" default="$(find ur_description)/config/$(arg ur_type)/joint_limits.yaml"/>
+   <xacro:property name="kinematics_params" default="$(find ur_description)/config/$(arg ur_type)/default_kinematics.yaml"/>
+   <xacro:property name="physical_params" default="$(find ur_description)/config/$(arg ur_type)/physical_parameters.yaml"/>
+   <xacro:property name="visual_params" default="$(find ur_description)/config/$(arg ur_type)/visual_parameters.yaml"/>
    <xacro:arg name="transmission_hw_interface" default=""/>
    <xacro:arg name="safety_limits" default="false"/>

Commit message: fix: try to make value constant

File: src/custom-ur-descriptions/ur3e_hande_robot_description/urdf/ur_with_hande.xacro (robot description, xacro)
@@ -12,8 +12,8 @@
    <!-- These parameters are from https://github.com/UniversalRobots/Universal_Robots_ROS2_Description/blob/29e90d5095fdf4af99eba3c3eae153d7d5d769c0/urdf/ur.urdf.xacro-->
    <xacro:arg name="tf_prefix" default="" />
-   <xacro:property name="joint_limit_params" default="$(find ur_description)/config/$(arg ur_type)/joint_limits.yaml"/>
-   <xacro:property name="kinematics_params" default="$(find ur_description)/config/$(arg ur_type)/default_kinematics.yaml"/>
-   <xacro:property name="physical_params" default="$(find ur_description)/config/$(arg ur_type)/physical_parameters.yaml"/>
-   <xacro:property name="visual_params" default="$(find ur_description)/config/$(arg ur_type)/visual_parameters.yaml"/>
+   <xacro:property name="joint_limit_params" value="$(find ur_description)/config/$(arg ur_type)/joint_limits.yaml"/>
+   <xacro:property name="kinematics_params" value="$(find ur_description)/config/$(arg ur_type)/default_kinematics.yaml"/>
+   <xacro:property name="physical_params" value="$(find ur_description)/config/$(arg ur_type)/physical_parameters.yaml"/>
+   <xacro:property name="visual_params" value="$(find ur_description)/config/$(arg ur_type)/visual_parameters.yaml"/>
    <xacro:arg name="transmission_hw_interface" default=""/>
    <xacro:arg name="safety_limits" default="false"/>

Commit message: fix: backward compatability

File: src/custom-ur-descriptions/ur3e_hande_robot_description/urdf/ur_with_hande.xacro (robot description, xacro)
@@ -12,8 +12,8 @@
    <!-- These parameters are from https://github.com/UniversalRobots/Universal_Robots_ROS2_Description/blob/29e90d5095fdf4af99eba3c3eae153d7d5d769c0/urdf/ur.urdf.xacro-->
    <xacro:arg name="tf_prefix" default="" />
-   <xacro:property name="joint_limit_params" value="$(find ur_description)/config/$(arg ur_type)/joint_limits.yaml"/>
-   <xacro:property name="kinematics_params" value="$(find ur_description)/config/$(arg ur_type)/default_kinematics.yaml"/>
-   <xacro:property name="physical_params" value="$(find ur_description)/config/$(arg ur_type)/physical_parameters.yaml"/>
-   <xacro:property name="visual_params" value="$(find ur_description)/config/$(arg ur_type)/visual_parameters.yaml"/>
+   <xacro:arg name="joint_limit_params" default="$(find ur_description)/config/$(arg ur_type)/joint_limits.yaml"/>
+   <xacro:arg name="kinematics_params" default="$(find ur_description)/config/$(arg ur_type)/default_kinematics.yaml"/>
+   <xacro:arg name="physical_params" default="$(find ur_description)/config/$(arg ur_type)/physical_parameters.yaml"/>
+   <xacro:arg name="visual_params" default="$(find ur_description)/config/$(arg ur_type)/visual_parameters.yaml"/>
    <xacro:arg name="transmission_hw_interface" default=""/>
    <xacro:arg name="safety_limits" default="false"/>
