Commit message: Add pipettor config, robot calibration, and kinematics tuning
- Add config/ur5e_calibration.yaml for robot-specific kinematics
- Add ur_with_zivid_pipettor description and MoveIt config
- Increase kinematics solver timeout (0.1→1.0s) and attempts (3→10)
- Update launch files with use_fake_hardware argument
- Update documentation

File: src/custom-ur-descriptions/ur5e_robot_description/urdf/te_robotside.xacro (robot description, xacro)
@@ -1,5 +1,5 @@
 <?xml version="1.0"?>
 <robot xmlns:xacro="http://ros.org/wiki/xacro" name="wingman_toolchanger_robotside">
-  <xacro:macro name="te_robotside" params="parent_link xyz:='0.010 0 0' rpy:='0 0 ${pi/2}'">
+  <xacro:macro name="te_robotside" params="parent_link xyz:='0.010 0 0' rpy:='0 0 ${pi/2}' scale:='0.001' mass:='0.5'">
     <link name="te_robotside">
       <visual>
@@ -7,5 +7,5 @@
         <geometry>
           <mesh filename="package://ur5e_robot_description/meshes/tool_exchanger/Tool_block_robotside.stl"
-                scale="0.001 0.001 0.001"/>
+                scale="${scale} ${scale} ${scale}"/>
         </geometry>
         <material name="grey">
@@ -17,9 +17,9 @@
         <geometry>
           <mesh filename="package://ur5e_robot_description/meshes/tool_exchanger/Tool_block_robotside.stl"
-                scale="0.001 0.001 0.001"/>
+                scale="${scale} ${scale} ${scale}"/>
         </geometry>
       </collision>
       <inertial>
-        <mass value="0.5"/>
+        <mass value="${mass}"/>
         <origin xyz="0 0 0" rpy="0 0 0"/>
         <inertia ixx="0.001" ixy="0.0" ixz="0.0"

File: src/custom-ur-descriptions/ur5e_robot_description/urdf/ur_standalone.xacro (robot description, xacro)
@@ -32,4 +32,6 @@
    <xacro:arg name="script_sender_port" default="50002"/>
    <xacro:arg name="trajectory_port" default="50003"/>
+   <!-- Keep-alive: number of 20ms cycles without response before disconnect (10 = 200ms timeout) -->
+   <xacro:arg name="keep_alive_count" default="10"/>
    <!--   tool communication related parameters-->
    <xacro:arg name="use_tool_communication" default="false" />
@@ -92,12 +94,14 @@
      script_sender_port="$(arg script_sender_port)"
      trajectory_port="$(arg trajectory_port)"
+     keep_alive_count="$(arg keep_alive_count)"
      >
      <origin xyz="0 0 0" rpy="0 0 0" />          <!-- position robot in the map -->
    </xacro:ur_robot>
   <!-- Modular Zivid: Arm Mount + Camera (with calibrated camera position) -->
+  <!-- Using tool0 instead of flange - Zivid calibration uses tool0 frame -->
   <xacro:zivid_camera_mount
-    parent_link="$(arg tf_prefix)flange"
-    xyz="0.005 0 0"
-    rpy="-1.5708 0 -1.5708"
+    parent_link="$(arg tf_prefix)tool0"
+    xyz="0 0 0.005"
+    rpy="0 0 3.14159"
     zivid_model="ZIVID_2_PLUS_MR60"/>
   <!-- Tool exchanger robotside attached to arm mount (not camera) -->

File: src/custom-ur-descriptions/ur5e_robot_description/urdf/ur_with_zivid_epick.urdf (robot description, URDF)
Before this commit: robot ur, 21 links, 20 joints
Links:
- removed link zivid_camera
- added link zivid_arm_mount, mass 0.170; collision mesh filename=package://ur5e_robot_description/meshes/zivid/zivid_custom_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 scale=1.0 1.0 1.0; visual mesh filename=package://ur5e_robot_description/meshes/zivid/zivid_custom_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 scale=1.0 1.0 1.0
- added link zivid_base_link; collision mesh filename=package://zivid_description/meshes/collision/zivid_2_plus_c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; visual mesh filename=package://zivid_description/meshes/visual/zivid_2_plus.stl
- added link zivid_optical_frame
Joints:
- removed joint zivid_camera_mount_joint
- added joint mount_to_camera_joint: type fixed, parent zivid_arm_mount, child zivid_base_link, origin xyz=0.02803 0.07664 -0.04577 rpy=0.53964 -1.53712 -2.13794
- added joint zivid_arm_mount_joint: type fixed, parent tool0, child zivid_arm_mount, origin xyz=0 0 0.005 rpy=0 0 3.14159
- added joint zivid_uncalibrated_optical_joint: type fixed, parent zivid_base_link, child zivid_optical_frame, origin xyz=0.049 0.03202 0.0295 rpy=-1.5707963267948966 0 -1.6144295580947547
- joint tool_block_joint: origin xyz=0 -0.105 0.03 rpy=-1.5708 0 0 -> xyz=0 0 0.055 rpy=-1.5708 0 3.14159; parent zivid_camera -> zivid_arm_mount

File: src/custom-ur-descriptions/ur5e_robot_description/urdf/ur_with_zivid_epick.xacro (robot description, xacro)
@@ -33,4 +33,6 @@
   <xacro:arg name="script_sender_port" default="50002"/>
   <xacro:arg name="trajectory_port" default="50003"/>
+  <!-- Keep-alive: number of 20ms cycles without response before disconnect (10 = 200ms timeout) -->
+  <xacro:arg name="keep_alive_count" default="10"/>
   <!-- tool communication related parameters -->
   <xacro:arg name="use_tool_communication" default="false" />
@@ -92,17 +94,19 @@
     script_sender_port="$(arg script_sender_port)"
     trajectory_port="$(arg trajectory_port)"
+    keep_alive_count="$(arg keep_alive_count)"
     >
     <origin xyz="0 0 0" rpy="0 0 0" />
   </xacro:ur_robot>
   <!-- Modular Zivid: Arm Mount + Camera (with calibrated camera position) -->
+  <!-- Using tool0 instead of flange - Zivid calibration uses tool0 frame -->
   <xacro:zivid_camera_mount
-    parent_link="$(arg tf_prefix)flange"
-    xyz="0.005 0 0"
-    rpy="-1.5708 0 -1.5708"
+    parent_link="$(arg tf_prefix)tool0"
+    xyz="0 0 0.005"
+    rpy="0 0 3.14159"
     zivid_model="ZIVID_2_PLUS_MR60"/>
   <!-- Tool block attached to the Zivid arm mount (not the camera) -->
   <xacro:tool_block parent_link="zivid_arm_mount" xyz="0 0 0.055" rpy="-1.5708 0 3.14159"/>
-  <!-- ZEpick Gripper -->
-  <xacro:epick_overlay use_fake_hardware="true" parent="tool_block"
+  <!-- Epick Gripper -->
+  <xacro:epick_overlay use_fake_hardware="$(arg use_fake_hardware)" parent="tool_block"
                   origin_xyz="0 -0.02 0"
                   origin_rpy="-1.5708 0 3.1416"/>

File: src/custom-ur-descriptions/ur5e_robot_description/urdf/ur_with_zivid_hande.urdf (robot description, URDF)
Before this commit: robot ur, 20 links, 19 joints
Links:
- removed link zivid_camera
- added link zivid_arm_mount, mass 0.170; collision mesh filename=package://ur5e_robot_description/meshes/zivid/zivid_custom_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 scale=1.0 1.0 1.0; visual mesh filename=package://ur5e_robot_description/meshes/zivid/zivid_custom_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 scale=1.0 1.0 1.0
- added link zivid_base_link; collision mesh filename=package://zivid_description/meshes/collision/zivid_2_plus_c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; visual mesh filename=package://zivid_description/meshes/visual/zivid_2_plus.stl
- added link zivid_optical_frame
Joints:
- removed joint zivid_camera_mount_joint
- added joint mount_to_camera_joint: type fixed, parent zivid_arm_mount, child zivid_base_link, origin xyz=0.02803 0.07664 -0.04577 rpy=0.53964 -1.53712 -2.13794
- added joint zivid_arm_mount_joint: type fixed, parent tool0, child zivid_arm_mount, origin xyz=0.00000 0.00000 0.00500 rpy=0.00000 0.00000 3.14159
- added joint zivid_uncalibrated_optical_joint: type fixed, parent zivid_base_link, child zivid_optical_frame, origin xyz=0.049 0.03202 0.0295 rpy=-1.5707963267948966 0 -1.6144295580947547
- joint tool_block_joint: origin xyz=0 -0.105 0.03 rpy=-1.5708 0 0 -> xyz=0 0 0.055 rpy=-1.5708 0 3.14159; parent zivid_camera -> zivid_arm_mount

File: src/custom-ur-descriptions/ur5e_robot_description/urdf/ur_with_zivid_pipettor.urdf (robot description, URDF)
Before this commit: robot ur5e, 17 links, 16 joints
Links:
- removed link te_robotside
- added link led_strip_link; visual box size=0.002 0.001 0.02
- added link pipette_base_link
- added link pipette_body_link, mass 0.2; collision mesh filename=package://pipette_description/meshes/collision/pipettor_col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 scale=0.001 0.001 0.001; visual mesh filename=package://pipette_description/meshes/visual/pipettor_visual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 scale=0.001 0.001 0.001
- added link pipette_tip_link
- added link tool_block, mass 0.2; collision mesh filename=package://ur5e_robot_description/meshes/tool_exchanger/Tool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 scale=0.001 0.001 0.001; visual mesh filename=package://ur5e_robot_description/meshes/tool_exchanger/Tool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 scale=0.001 0.001 0.001
Joints:
- removed joint te_robotside_joint
- added joint led_strip_joint: type fixed, parent pipette_base_link, child led_strip_link, origin xyz=0 0.025 0.238 rpy=0 0 0
- added joint pipette_attachment_joint: type fixed, parent tool_block, child pipette_base_link, origin xyz=-0.005 -0.015 0 rpy=-1.5708 0 3.1416
- added joint pipette_orientation_joint: type fixed, parent pipette_base_link, child pipette_body_link, origin xyz=-0.09 -0.055 0.34 rpy=-1.5708 0 0
- added joint pipette_tip_joint: type fixed, parent pipette_base_link, child pipette_tip_link, origin xyz=0 0 0.34 rpy=0 0 0
- added joint tool_block_joint: type fixed, parent zivid_arm_mount, child tool_block, origin xyz=0 0 0.055 rpy=-1.5708 0 3.14159

File: src/custom-ur-descriptions/ur5e_robot_description/urdf/ur_with_zivid_pipettor.xacro (robot description, xacro)
@@ -1,5 +1,5 @@
 <?xml version="1.0"?>
 <robot xmlns:xacro="http://wiki.ros.org/xacro" name="$(arg name)">
-<!--Chain: map -> UR -> flange -> zivid_camera_mount -> zivid_camera -> HandE gripper -->
+<!--Chain: map -> UR -> flange -> zivid_camera_mount -> zivid_camera -> tool_block -> pipettor -->
   <!-- robot name parameter -->
   <xacro:arg name="name" default="ur5e"/>
@@ -8,5 +8,5 @@
   <xacro:include filename="$(find ur5e_robot_description)/urdf/zivid_camera_mount.xacro"/>
   <xacro:include filename="$(find ur5e_robot_description)/urdf/tool_block.xacro"/>
-  <xacro:include filename="$(find robotiq_hande_description)/urdf/robotiq_hande_gripper.xacro"/>
+  <xacro:include filename="$(find pipette_description)/urdf/pipette_macro.urdf.xacro"/>
   <!-- possible 'ur_type' values: ur3, ur5e, ur5, ur10, ur10e, ur16e, ur20 -->
   <xacro:arg name="ur_type" default="ur5e"/>
@@ -35,6 +35,6 @@
   <xacro:arg name="keep_alive_count" default="10"/>
   <!-- tool communication related parameters -->
-  <xacro:arg name="use_tool_communication" default="false" />
-  <xacro:arg name="tool_voltage" default="0" />
+  <xacro:arg name="use_tool_communication" default="true" />
+  <xacro:arg name="tool_voltage" default="24" />
   <xacro:arg name="tool_parity" default="0" />
   <xacro:arg name="tool_baud_rate" default="115200" />
@@ -101,39 +101,17 @@
   <xacro:zivid_camera_mount
     parent_link="$(arg tf_prefix)tool0"
-    xyz="0.00000 0.00000 0.00500"
-    rpy="0.00000 0.00000 3.14159"
+    xyz="0 0 0.005"
+    rpy="0 0 3.14159"
     zivid_model="ZIVID_2_PLUS_MR60"/>
   <!-- Tool block attached to the Zivid arm mount (not the camera) -->
   <xacro:tool_block parent_link="zivid_arm_mount" xyz="0 0 0.055" rpy="-1.5708 0 3.14159"/>
-  <!-- gripper pos wrt camera    -->
-  <xacro:arg name="grip_pos_min" default="0"/>
-  <xacro:arg name="grip_pos_max" default="0.025"/>
-  <xacro:arg name="tty_port" default="/tmp/ttyUR"/>
-  <xacro:arg name="baudrate" default="115200"/>
-  <xacro:arg name="parity" default="N"/>
-  <xacro:arg name="data_bits" default="8"/>
-  <xacro:arg name="stop_bit" default="1"/>
-  <xacro:arg name="slave_id" default="9"/>
-  <xacro:arg name="create_socat_tty" default="true"/>
-  <xacro:arg name="socat_ip_address" default="$(arg robot_ip)"/>
-  <xacro:arg name="socat_port" default="54321"/>
-  <xacro:robotiq_hande_gripper
-    name="robotiq_hande_gripper"
+  <!-- Pipettor attached to tool block -->
+  <xacro:pipette
+    name="pipette"
     prefix="$(arg tf_prefix)"
     parent="tool_block"
-    grip_pos_min="$(arg grip_pos_min)"
-    grip_pos_max="$(arg grip_pos_max)"
-    tty_port="$(arg tty_port)"
-    baudrate="$(arg baudrate)"
-    parity="$(arg parity)"
-    data_bits="$(arg data_bits)"
-    stop_bit="$(arg stop_bit)"
-    slave_id="$(arg slave_id)"
-    use_fake_hardware="$(arg use_fake_hardware)"
-    xyz="0 -0.02 0"
+    pipette_mass="0.200"
+    xyz="-0.005 -0.015 0"
     rpy="-1.5708 0 3.1416"
-    create_socat_tty="$(arg create_socat_tty)"
-    socat_ip_address="$(arg socat_ip_address)"
-    socat_port="$(arg socat_port)"
   />
 </robot>

File: src/custom-ur-descriptions/ur5e_robot_description/urdf/zivid_camera_mount.xacro (robot description, xacro)
@@ -43,13 +43,11 @@
       model="${zivid_model}"
       field_of_view="false"/>
-    <!-- Joint: Arm Mount -> Camera                   -->
-    <!-- CALIBRATION: Adjust xyz/rpy to match setup   -->
+    <!-- Joint: Arm Mount -> Camera Base Link -->
+    <!-- Zivid calibration uses tool0 frame per: https://github.com/zivid/zivid-ros/issues/124 -->
     <joint name="mount_to_camera_joint" type="fixed">
       <parent link="zivid_arm_mount"/>
       <child link="zivid_base_link"/>
-      <!-- for forward mounted camera bracket -->
-            <!-- <origin xyz="0.025 0.062 0.0" rpy="0 -1.5708 -1.5708"/> -->
-      <!-- for backward mounted camera bracket -->
-      <origin xyz="0.025 0.062 -0.049" rpy="0 -1.5708 -1.5708"/>
+      <origin xyz="0.02803 0.07664 -0.04577"
+              rpy="0.53964 -1.53712 -2.13794"/>
     </joint>
   </xacro:macro>
